File: circuit/twpc.sch (EAGLE design)
At the start: 2 parts

Commit message: New circuit
Hopefully the final
Parts:
- added Q1: NDP6020P, transistor-power:PMOSFET_PTO220BH
- R1: value 4K7 -> 2K2; device resistor:R-US_0204/7 -> resistor:R-US_0204/5
- R2: device resistor:R-US_0204/7 -> resistor:R-US_0204/2V
Connections:
- net 0V renamed GND
- new net +5V: Q1.S
- new net N$2: Q1.D, R1.2, R2.2
- net N$1: now also Q1.G; no longer R1.2, R2.2
Other:
- note added: "RAILS"
- note added: "TWPC_DATA_P"
- note added: "TWPC_POWER_P"
- note added: "device"
- note added: "master"
- note removed: "Metal contacts"
- note removed: "ONEWIRE_P"
- note removed: "onewire_pins[]"
- note removed: "station"
- note removed: "train"
- moved on the sheet: R1, R2
Changed lines of the file:
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@@
 <grid distance="0.1" unitdist="inch" unit="inch" style="lines" multiple="1" display="no" altdistance="0.01" altunitdist="inch" altunit="inch"/>
 <layers>
-<layer number="1" name="Top" color="4" fill="1" visible="no" active="no"/>
+<layer number="1" name="Top" color="4" fill="11" visible="no" active="no"/>
 <layer number="16" name="Bottom" color="1" fill="1" visible="no" active="no"/>
 <layer number="17" name="Pads" color="2" fill="1" visible="no" active="no"/>
@@
 <layer number="48" name="Document" color="7" fill="1" visible="no" active="no"/>
 <layer number="49" name="Reference" color="7" fill="1" visible="no" active="no"/>
-<layer number="51" name="tDocu" color="7" fill="1" visible="no" active="no"/>
+<layer number="51" name="tDocu" color="6" fill="1" visible="no" active="no"/>
 <layer number="52" name="bDocu" color="7" fill="1" visible="no" active="no"/>
 <layer number="91" name="Nets" color="2" fill="1" visible="yes" active="yes"/>
@@
 </classes>
 <parts>
-<part name="R1" library="resistor" deviceset="R-US_" device="0204/7" value="4K7"/>
-<part name="R2" library="resistor" deviceset="R-US_" device="0204/7" value="10K"/>
-<part name="GND1" library="supply1" deviceset="0V" device=""/>
-<part name="GND2" library="supply1" deviceset="0V" device=""/>
+<part name="Q1" library="transistor-power" deviceset="PMOSFET_P" device="TO220BH" value="NDP6020P"/>
+<part name="P+1" library="supply1" deviceset="+5V" device=""/>
+<part name="GND1" library="supply1" deviceset="GND" device=""/>
 <part name="SUPPLY1" library="supply2" deviceset="V--&gt;" device=""/>
-<part name="SUPPLY2" library="supply2" deviceset="V&lt;--" device=""/>
+<part name="SUPPLY2" library="supply2" deviceset="V--&gt;" device=""/>
+<part name="SUPPLY3" library="supply2" deviceset="V&lt;--" device=""/>
+<part name="R1" library="resistor" deviceset="R-US_" device="0204/5" value="2K2"/>
+<part name="R2" library="resistor" deviceset="R-US_" device="0204/2V" value="10K"/>
+<part name="GND2" library="supply1" deviceset="GND" device=""/>
 </parts>
 <sheets>
 <sheet>
 <plain>
-<text x="33.02" y="68.58" size="1.778" layer="97">ONEWIRE_P</text>
-<text x="-30.48" y="68.58" size="1.778" layer="97">onewire_pins[]</text>
-<text x="0" y="66.04" size="1.778" layer="97">Metal contacts</text>
-<text x="-27.94" y="60.96" size="1.778" layer="97">station</text>
-<text x="38.1" y="60.96" size="1.778" layer="97">train</text>
+<text x="-1859.28" y="660.4" size="1.778" layer="97">TWPC_POWER_P</text>
+<text x="-1859.28" y="647.7" size="1.778" layer="97">TWPC_DATA_P</text>
+<text x="-1783.08" y="647.7" size="1.778" layer="97">TWPC_DATA_P</text>
+<text x="-1856.74" y="652.78" size="1.778" layer="97">master</text>
+<text x="-1778" y="640.08" size="1.778" layer="97">device</text>
+<text x="-1813.56" y="645.16" size="1.778" layer="97">RAILS</text>
 </plain>
 <instances>
-<instance part="R1" gate="G$1" x="-7.62" y="58.42" rot="R90"/>
-<instance part="R2" gate="G$1" x="22.86" y="58.42" rot="R90"/>
-<instance part="GND1" gate="1" x="-7.62" y="45.72"/>
-<instance part="GND2" gate="1" x="22.86" y="45.72"/>
-<instance part="SUPPLY1" gate="G$1" x="-30.48" y="66.04"/>
-<instance part="SUPPLY2" gate="G$1" x="48.26" y="66.04"/>
+<instance part="Q1" gate="G$1" x="-1831.34" y="655.32"/>
+<instance part="P+1" gate="1" x="-1828.8" y="673.1"/>
+<instance part="GND1" gate="1" x="-1828.8" y="624.84"/>
+<instance part="SUPPLY1" gate="G$1" x="-1859.28" y="657.86"/>
+<instance part="SUPPLY2" gate="G$1" x="-1859.28" y="645.16"/>
+<instance part="SUPPLY3" gate="G$1" x="-1767.84" y="645.16"/>
+<instance part="R1" gate="G$1" x="-1828.8" y="637.54" rot="R90"/>
+<instance part="R2" gate="G$1" x="-1790.7" y="637.54" rot="R90"/>
+<instance part="GND2" gate="1" x="-1790.7" y="624.84"/>
 </instances>
 <busses>
@@
 <net name="N$1" class="0">
 <segment>
-<wire x1="-15.24" y1="66.04" x2="-7.62" y2="66.04" width="0.1524" layer="91"/>
-<pinref part="R1" gate="G$1" pin="2"/>
-<wire x1="33.02" y1="66.04" x2="22.86" y2="66.04" width="0.1524" layer="91"/>
-<wire x1="22.86" y1="66.04" x2="-7.62" y2="66.04" width="0.1524" layer="91"/>
-<wire x1="-7.62" y1="66.04" x2="-7.62" y2="63.5" width="0.1524" layer="91"/>
-<pinref part="R2" gate="G$1" pin="2"/>
-<wire x1="22.86" y1="66.04" x2="22.86" y2="63.5" width="0.1524" layer="91"/>
-<junction x="22.86" y="66.04"/>
-<junction x="-7.62" y="66.04"/>
+<pinref part="Q1" gate="G$1" pin="G"/>
+<wire x1="-1844.04" y1="657.86" x2="-1836.42" y2="657.86" width="0.1524" layer="91"/>
 </segment>
 </net>
-<net name="0V" class="0">
+<net name="+5V" class="0">
+<segment>
+<pinref part="Q1" gate="G$1" pin="S"/>
+<pinref part="P+1" gate="1" pin="+5V"/>
+<wire x1="-1828.8" y1="660.4" x2="-1828.8" y2="670.56" width="0.1524" layer="91"/>
+</segment>
+</net>
+<net name="N$2" class="0">
+<segment>
+<pinref part="Q1" gate="G$1" pin="D"/>
+<pinref part="R1" gate="G$1" pin="2"/>
+<wire x1="-1828.8" y1="650.24" x2="-1828.8" y2="645.16" width="0.1524" layer="91"/>
+<wire x1="-1828.8" y1="645.16" x2="-1828.8" y2="642.62" width="0.1524" layer="91"/>
+<wire x1="-1783.08" y1="645.16" x2="-1790.7" y2="645.16" width="0.1524" layer="91"/>
+<junction x="-1828.8" y="645.16"/>
+<wire x1="-1790.7" y1="645.16" x2="-1828.8" y2="645.16" width="0.1524" layer="91"/>
+<wire x1="-1828.8" y1="645.16" x2="-1844.04" y2="645.16" width="0.1524" layer="91"/>
+<pinref part="R2" gate="G$1" pin="2"/>
+<wire x1="-1790.7" y1="642.62" x2="-1790.7" y2="645.16" width="0.1524" layer="91"/>
+<junction x="-1790.7" y="645.16"/>
+</segment>
+</net>
+<net name="GND" class="0">
 <segment>
 <pinref part="R1" gate="G$1" pin="1"/>
-<pinref part="GND1" gate="1" pin="0V"/>
-<wire x1="-7.62" y1="53.34" x2="-7.62" y2="48.26" width="0.1524" layer="91"/>
+<pinref part="GND1" gate="1" pin="GND"/>
+<wire x1="-1828.8" y1="632.46" x2="-1828.8" y2="627.38" width="0.1524" layer="91"/>
 </segment>
 <segment>
 <pinref part="R2" gate="G$1" pin="1"/>
-<pinref part="GND2" gate="1" pin="0V"/>
-<wire x1="22.86" y1="53.34" x2="22.86" y2="48.26" width="0.1524" layer="91"/>
+<pinref part="GND2" gate="1" pin="GND"/>
+<wire x1="-1790.7" y1="632.46" x2="-1790.7" y2="627.38" width="0.1524" layer="91"/>
 </segment>
 </net>
@@
 </sheet>
 </sheets>
+<errors>
+</errors>
 </schematic>
 </drawing>
